File: kicad/v3/rgb-to-hdmi.kicad_pcb (KiCad board)
At the start: 2 copper layers, 65 x 30 mm, 31 parts, among them P1 CONN_02X20, P2 CONN_01X03, P3 CONN_01X06, P4 CONN_01X02, P5 CONN_01X06, P6 CONN_01X02, P7 Conn_01x01, SW1 SW_PUSH, SW2 SW_PUSH, SW3 SW_PUSH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

Commit message: KiCad: increased via size from 24 to 26 mil
Change-Id: I74ec79289cb28377dae48824100bb691867bed43
Routing:
- net /GPIO25: track 79.7 -> 81.4 mm
- net /GPIO16: track 60.6 -> 62.0 mm
- net /GPIO26: track 50.7 -> 51.5 mm
Other:
- net class Default: via_dia 0.6096 -> 0.6604
- net class Power: via_dia 0.6096 -> 0.762; via_drill 0.3048 -> 0.381
- rule via_min_size: 0.6096 -> 0.6604

Commit message: KiCad: final cleanup phase
Change-Id: I2b417b60cc912d6b221c863d25bd544ac01c97df
Parts:
- moved SW4 0.38 mm to (76.1, 36.9)
- moved P6 0.23 mm to (66.5, 41.4)
Other:
- rule pad_to_mask_clearance: 0.2 -> 0.15
