File: kicad_analog/V2/analog.kicad_pcb (KiCad board)
At the start: 2 copper layers, 50 x 23.2 mm, 32 parts, among them P1 Conn_02x05_Odd_Even, P2 Conn_01x04, P3 Conn_01x06, P4 Conn_01x02, P6 Conn_01x01, P7 Conn_01x01, U1 MAX9144, U2 MAX9144, U3 4066, U4 MAX5259EEE+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

Commit message: Issue 2 analog board part2
Parts:
- moved C1 0.15 mm to (35.9, 52.3)
- moved C2 0.15 mm to (38.5, 52.3)
- moved C4 0.15 mm to (41.3, 52.3)
- moved Cx2 0.08 mm to (39.8, 47.3)
Routing:
- net /VSYNC: track 10.3 -> 11.0 mm
Other:
- board text added: "DAC:"
- board text added: "MAX5259"
- board text added: "MAX5259 DAC Issue 2 ©2019 IanB"
- board text removed: "MAX9108"
- board text removed: "MAX9108 / MAX9144 Issue 2 ©2019 IanB"
- board text removed: "MAX9144"
