File: Kicad_6Bit/v3/rgb-to-hdmi.kicad_pcb (KiCad board)
At the start: 2 copper layers, 65 x 30 mm, 40 parts, among them J2 Conn_02x01, P1 CONN_02X20, P2 Conn_02x05_Odd_Even, P3 Conn_01x06, P4 CONN_01X02, P5 Conn_01x04, SW1 SW_PUSH, SW2 SW_PUSH, SW3 SW_PUSH, SW4 SW_PUSH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

Commit message: Update V3 hat pcb
Parts:
- added JP6: SolderJumper_2_Bridged, Jumper:SolderJumper-2_P1.3mm_Bridged_RoundedPad1.0x1.5mm, F.Cu at (59.6, 44.8)
- moved JP5 0.28 mm to (37.7, 52.8)
Connections:
- JP5 pad 1: /UV1 -> /UV3
- JP5 pad 2: /UV3 -> /GPIO26
- U1 pad 21: /GPIO27 -> /UV4
Routing:
- net /DETECT: track 85.7 -> 52.7 mm, vias 4 -> 2
- net /UV4: track 0.00 -> 29.6 mm, vias 0 -> 2
- net /GPIO26: track 46.2 -> 59.3 mm
- net /GPIO19: track 31.8 -> 40.2 mm
- net /GPIO27: track 60.0 -> 53.7 mm
- net /UV1: track 43.6 -> 39.0 mm
- net /UV3: track 11.6 -> 16.1 mm
- net /GPIO1: track 42.7 -> 44.2 mm
- net /TDO: track 54.3 -> 55.7 mm
Other:
- board text added: "1"
