File: Kicad_6Bit/v3/rgb-to-hdmi.sch (KiCad schematic (older format))
At the start: 30 parts, among them J2 Conn_02x01, P1 CONN_02X20, P2 Conn_02x05_Odd_Even, P3 Conn_01x06, P4 CONN_01X02, P5 Conn_01x04, SW1 SW_PUSH, SW2 SW_PUSH, SW3 SW_PUSH, SW4 SW_PUSH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

Commit message: Update V3 hat pcb
Parts:
- added JP6: SolderJumper_2_Bridged, Jumper:SolderJumper-2_P1.3mm_Bridged_RoundedPad1.0x1.5mm, symbol Jumper:SolderJumper_2_Bridged
Connections:
- net GPIO19: now also JP6.2 (B)
- net GPIO26: now also JP5.2 (B)
- net GPIO27: no longer U1.21 (F4M8)
- net UV1: no longer JP5.1 (A)
- net UV3: now also JP5.1 (A); no longer JP5.2 (B)
- new net UV4: JP6.1 (A), U1.21 (F4M8)
Other:
- moved on the sheet: JP5
