File: Kicad_6Bit/v3_Template/rgb-to-hdmi.kicad_pcb (KiCad board)
At the start: 2 copper layers, 67.6 x 30.5 mm, 41 parts, among them J2 Conn_02x01, P1 CONN_02X20, P2 Conn_02x05_Odd_Even, P3 Conn_01x06, P4 CONN_01X02, P5 Conn_01x04, SW1 SW_PUSH, SW2 SW_PUSH, SW3 SW_PUSH, SW4 SW_PUSH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

Commit message: Update 6/8 bit pcbs
Parts:
- D1, D2: footprint LED_THT:LED_D1.8mm_W3.3mm_H2.4mm -> LED_THT:LED_D1.8mm_W3.3mm_H2.4mm_Custom
- P1: footprint Connector_PinSocket_2.54mm:PinSocket_2x20_P2.54mm_Vertical -> Connector_PinSocket_2.54mm:PinSocket_2x20_P2.54mm_Vertical_Custom
- P4: footprint Connector_PinSocket_2.54mm:PinSocket_1x02_P2.54mm_Vertical -> Connector_PinSocket_2.54mm:PinSocket_1x02_P2.54mm_Vertical_Custom
- renumbered JP5 to X3, JP6 to X4
Connections:
- net /UV1 renamed /X1
- net /UV2 renamed /X2
- net /UV3 renamed /X3
- net /UV4 renamed /X4
Routing:
- net /GPIO27: track 53.7 -> 52.9 mm
- net Net-(D1-Pad1): track 4.28 -> 3.66 mm
Other:
- board text added: "X1"
- board text added: "X2"
- board text removed: "1"

Commit message: Update gerbers
Parts:
- renumbered X3 to JP5, X4 to JP6
Changed lines of the file:
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@@
     (tags "solder jumper open")
     (attr virtual)
-    (fp_text reference X3 (at -2.20496 0.08976) (layer F.SilkS)
+    (fp_text reference JP5 (at -2.55512 0.09652) (layer F.SilkS)
       (effects (font (size 0.8 0.8) (thickness 0.12)))
     )
@@
     (tags "solder jumper open")
     (attr virtual)
-    (fp_text reference X4 (at -2.182 0.08818) (layer F.SilkS)
+    (fp_text reference JP6 (at -2.63386 0.11176) (layer F.SilkS)
       (effects (font (size 0.8 0.8) (thickness 0.12)))
     )
@@
   (segment (start 34.532 26.73096) (end 34.532 27.23896) (width 0.2032) (layer F.Cu) (net 46) (status 30))
   (segment (start 31.992 26.73096) (end 31.992 27.23896) (width 0.2032) (layer F.Cu) (net 47) (status 30))
+  (segment (start 70.092 45.75556) (end 71.87 45.75556) (width 0.2032) (layer F.Cu) (net 48) (status 10))
+  (segment (start 72.1494 46.03496) (end 71.87 45.75556) (width 0.2032) (layer F.Cu) (net 48))
+  (segment (start 74.8582 46.03496) (end 72.1494 46.03496) (width 0.2032) (layer F.Cu) (net 48))
+  (segment (start 69.242001 46.605559) (end 69.242001 49.079519) (width 0.2032) (layer F.Cu) (net 48))
+  (segment (start 70.092 45.75556) (end 69.242001 46.605559) (width 0.2032) (layer F.Cu) (net 48))
+  (segment (start 67.84156 50.47996) (end 66.6122 50.47996) (width 0.2032) (layer F.Cu) (net 48))
+  (segment (start 69.242001 49.079519) (end 67.84156 50.47996) (width 0.2032) (layer F.Cu) (net 48))
+  (via (at 44.480526 32.228921) (size 0.6604) (drill 0.3048) (layers F.Cu B.Cu) (net 48))
+  (segment (start 44.362 32.347447) (end 44.480526 32.228921) (width 0.2032) (layer F.Cu) (net 48))
+  (segment (start 44.362 33.76846) (end 44.362 32.347447) (width 0.2032) (layer F.Cu) (net 48))
+  (segment (start 44.480526 32.228921) (end 44.480526 32.774861) (width 0.2032) (layer B.Cu) (net 48))
+  (segment (start 44.480526 32.774861) (end 45.078715 33.37305) (width 0.2032) (layer B.Cu) (net 48))
+  (segment (start 60.00058 44.29577) (end 64.86397 44.29577) (width 0.2032) (layer B.Cu) (net 48))
+  (segment (start 56.07952 40.62221) (end 52.85372 40.62221) (width 0.2032) (layer B.Cu) (net 48))
+  (via (at 64.99676 44.16298) (size 0.6604) (drill 0.3048) (layers F.Cu B.Cu) (net 48))
+  (segment (start 52.85372 40.62221) (end 52.17739 39.94588) (width 0.2032) (layer B.Cu) (net 48))
+  (segment (start 64.86397 44.29577) (end 64.99676 44.16298) (width 0.2032) (layer B.Cu) (net 48))
+  (segment (start 52.17739 39.94588) (end 52.177389 34.365499) (width 0.2032) (layer B.Cu) (net 48))
+  (segment (start 52.177389 34.365499) (end 51.18494 33.37305) (width 0.2032) (layer B.Cu) (net 48))
+  (segment (start 66.6122 50.47996) (end 66.02038 49.88814) (width 0.2032) (layer F.Cu) (net 48))
+  (segment (start 60.00058 44.29577) (end 56.32702 40.62221) (width 0.2032) (layer B.Cu) (net 48))
+  (segment (start 56.32702 40.62221) (end 52.85372 40.62221) (width 0.2032) (layer B.Cu) (net 48))
+  (segment (start 45.078715 33.37305) (end 51.184941 33.373051) (width 0.2032) (layer B.Cu) (net 48))
+  (segment (start 65.97466 49.84242) (end 66.02038 49.88814) (width 0.2032) (layer F.Cu) (net 48))
+  (segment (start 64.99676 44.16298) (end 65.97466 45.14088) (width 0.2032) (layer F.Cu) (net 48))
+  (segment (start 65.97466 45.14088) (end 65.97466 49.84242) (width 0.2032) (layer F.Cu) (net 48))
   (segment (start 20.572358 47.05096) (end 20.1048 46.583402) (width 0.2032) (layer F.Cu) (net 49))
   (segment (start 24.372 47.05096) (end 20.572358 47.05096) (width 0.2032) (layer F.Cu) (net 49))
@@
   (segment (start 41.09282 50.92446) (end 40.75009 51.26719) (width 0.2032) (layer F.Cu) (net 51))
   (segment (start 40.75009 51.26719) (end 39.66805 51.26719) (width 0.2032) (layer F.Cu) (net 51))
-  (segment (start 70.092 45.75556) (end 71.87 45.75556) (width 0.2032) (layer F.Cu) (net 48) (status 10))
-  (segment (start 72.1494 46.03496) (end 71.87 45.75556) (width 0.2032) (layer F.Cu) (net 48))
-  (segment (start 74.8582 46.03496) (end 72.1494 46.03496) (width 0.2032) (layer F.Cu) (net 48))
-  (segment (start 69.242001 46.605559) (end 69.242001 49.079519) (width 0.2032) (layer F.Cu) (net 48))
-  (segment (start 70.092 45.75556) (end 69.242001 46.605559) (width 0.2032) (layer F.Cu) (net 48))
-  (segment (start 67.84156 50.47996) (end 66.6122 50.47996) (width 0.2032) (layer F.Cu) (net 48))
-  (segment (start 69.242001 49.079519) (end 67.84156 50.47996) (width 0.2032) (layer F.Cu) (net 48))
-  (via (at 44.480526 32.228921) (size 0.6604) (drill 0.3048) (layers F.Cu B.Cu) (net 48))
-  (segment (start 44.362 32.347447) (end 44.480526 32.228921) (width 0.2032) (layer F.Cu) (net 48))
-  (segment (start 44.362 33.76846) (end 44.362 32.347447) (width 0.2032) (layer F.Cu) (net 48))
-  (segment (start 44.480526 32.228921) (end 44.480526 32.774861) (width 0.2032) (layer B.Cu) (net 48))
-  (segment (start 44.480526 32.774861) (end 45.078715 33.37305) (width 0.2032) (layer B.Cu) (net 48))
-  (segment (start 60.00058 44.29577) (end 64.86397 44.29577) (width 0.2032) (layer B.Cu) (net 48))
-  (segment (start 56.07952 40.62221) (end 52.85372 40.62221) (width 0.2032) (layer B.Cu) (net 48))
-  (via (at 64.99676 44.16298) (size 0.6604) (drill 0.3048) (layers F.Cu B.Cu) (net 48))
-  (segment (start 52.85372 40.62221) (end 52.17739 39.94588) (width 0.2032) (layer B.Cu) (net 48))
-  (segment (start 64.86397 44.29577) (end 64.99676 44.16298) (width 0.2032) (layer B.Cu) (net 48))
-  (segment (start 52.17739 39.94588) (end 52.177389 34.365499) (width 0.2032) (layer B.Cu) (net 48))
-  (segment (start 52.177389 34.365499) (end 51.18494 33.37305) (width 0.2032) (layer B.Cu) (net 48))
-  (segment (start 66.6122 50.47996) (end 66.02038 49.88814) (width 0.2032) (layer F.Cu) (net 48))
-  (segment (start 60.00058 44.29577) (end 56.32702 40.62221) (width 0.2032) (layer B.Cu) (net 48))
-  (segment (start 56.32702 40.62221) (end 52.85372 40.62221) (width 0.2032) (layer B.Cu) (net 48))
-  (segment (start 45.078715 33.37305) (end 51.184941 33.373051) (width 0.2032) (layer B.Cu) (net 48))
-  (segment (start 65.97466 49.84242) (end 66.02038 49.88814) (width 0.2032) (layer F.Cu) (net 48))
-  (segment (start 64.99676 44.16298) (end 65.97466 45.14088) (width 0.2032) (layer F.Cu) (net 48))
-  (segment (start 65.97466 45.14088) (end 65.97466 49.84242) (width 0.2032) (layer F.Cu) (net 48))
   (via (at 43.05116 32.41294) (size 0.6604) (drill 0.3048) (layers F.Cu B.Cu) (net 52))
   (segment (start 42.762 33.76846) (end 42.762 32.7021) (width 0.2032) (layer F.Cu) (net 52))
