File: kicad_analog_6bit/V3 - Copy/analog.sch (KiCad schematic (older format))
At the start: 37 parts, among them P1 Conn_02x06_Odd_Even, P2 Conn_01x04, P3 Conn_01x06, P4 Conn_01x03_ODD, P5 Conn_01x03_EVEN, P6 Conn_01x01, P7 Conn_01x01, U1 MAX9108, U2 MAX9108, U3 TS12A44514DR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

Commit message: Extend P4 pads on analog board
Parts:
- P3: footprint Connector_Molex:Molex_PicoBlade_53048-0610_1x06_P1.25mm_Horizontal_Custom2 -> Connector_Molex:Molex_PicoBlade_53048-0610_1x06_P1.25mm_Horizontal
- P4: footprint Connector_Harwin:Harwin_M20-89003xx_1x03_P2.54mm_Horizontal_Custom_ODD -> Connector_Harwin:Harwin_M20-89003xx_1x03_P2.54mm_Horizontal_Custom_ODD2
- P5: footprint Connector_Harwin:Harwin_M20-89003xx_1x03_P2.54mm_Horizontal_Custom_EVEN -> Connector_Harwin:Harwin_M20-89003xx_1x03_P2.54mm_Horizontal_Custom_EVEN2
Changed lines of the file:
@@
 F 0 "P3" H 1368 925 50  0000 C CNN
 F 1 "Conn_01x06" H 1368 1016 50  0000 C CNN
-F 2 "Connector_Molex:Molex_PicoBlade_53048-0610_1x06_P1.25mm_Horizontal_Custom2" H 1450 1450 50  0001 C CNN
+F 2 "Connector_Molex:Molex_PicoBlade_53048-0610_1x06_P1.25mm_Horizontal" H 1450 1450 50  0001 C CNN
 F 3 "~" H 1450 1450 50  0001 C CNN
 	1    1450 1450
@@
 F 0 "P5" H 5050 4950 50  0000 C CNN
 F 1 "Conn_01x03_EVEN" H 4750 5050 50  0000 C CNN
-F 2 "Connector_Harwin:Harwin_M20-89003xx_1x03_P2.54mm_Horizontal_Custom_EVEN" H 5050 4700 50  0001 C CNN
+F 2 "Connector_Harwin:Harwin_M20-89003xx_1x03_P2.54mm_Horizontal_Custom_EVEN2" H 5050 4700 50  0001 C CNN
 F 3 "~" H 5050 4700 50  0001 C CNN
 	1    5050 4700
@@
 F 0 "P4" H 4850 4450 50  0000 L CNN
 F 1 "Conn_01x03_ODD" H 4300 4350 50  0000 L CNN
-F 2 "Connector_Harwin:Harwin_M20-89003xx_1x03_P2.54mm_Horizontal_Custom_ODD" H 4900 4700 50  0001 C CNN
+F 2 "Connector_Harwin:Harwin_M20-89003xx_1x03_P2.54mm_Horizontal_Custom_ODD2" H 4900 4700 50  0001 C CNN
 F 3 "~" H 4900 4700 50  0001 C CNN
 	1    4900 4700
