File: Kicad_6Bit/oldv3_Standard/rgb-to-hdmi.sch (KiCad schematic (older format))
At the start: 32 parts, among them J2 Conn_02x01, P1 CONN_02X20, P2 Conn_02x05_Odd_Even, P3 Conn_01x06, P4 CONN_01X02, P5 Conn_01x04, SW1 SW_PUSH, SW2 SW_PUSH, SW3 SW_PUSH, SW4 SW_PUSH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

Commit message: Update 6/8 bit boards with identity resistor
Parts:
- removed R7: 1K, Resistor_SMD:R_0805_2012Metric_Pad1.15x1.40mm_HandSolder, symbol Device:R_Small
- D1, D2: footprint LED_THT:LED_D1.8mm_W3.3mm_H2.4mm_Custom -> LED_THT:LED_D1.8mm_W3.3mm_H2.4mm
Changed lines of the file:
@@
 F 0 "D1" H 2000 3100 50  0000 C CNN
 F 1 "LED" H 2000 2900 50  0000 C CNN
-F 2 "LED_THT:LED_D1.8mm_W3.3mm_H2.4mm_Custom" H 2000 3000 50  0001 C CNN
+F 2 "LED_THT:LED_D1.8mm_W3.3mm_H2.4mm" H 2000 3000 50  0001 C CNN
 F 3 "" H 2000 3000 50  0001 C CNN
 	1    2000 3000
@@
 F 0 "D2" H 2300 3100 50  0000 C CNN
 F 1 "LED" H 2300 2900 50  0000 C CNN
-F 2 "LED_THT:LED_D1.8mm_W3.3mm_H2.4mm_Custom" H 2300 3000 50  0001 C CNN
+F 2 "LED_THT:LED_D1.8mm_W3.3mm_H2.4mm" H 2300 3000 50  0001 C CNN
 F 3 "" H 2300 3000 50  0001 C CNN
 	1    2300 3000
@@
 	1    0    0    -1
 $EndComp
-$Comp
-L Device:R_Small R7
-U 1 1 5E5AD207
-P 1850 2250
-F 0 "R7" H 1909 2296 50  0000 L CNN
-F 1 "1K" H 1909 2205 50  0000 L CNN
-F 2 "Resistor_SMD:R_0805_2012Metric_Pad1.15x1.40mm_HandSolder" H 1850 2250 50  0001 C CNN
-F 3 "~" H 1850 2250 50  0001 C CNN
-	1    1850 2250
-	1    0    0    -1
-$EndComp
-Wire Wire Line
-	1850 2000 1850 2150
-Text Label 1850 2450 0    60   ~ 0
-GND
-Wire Wire Line
-	1850 2450 1850 2350
 $EndSCHEMATC
