File: kicad_AmigaAdapter/V1/deniseadapter.sch (KiCad schematic (older format))
At the start: 14 parts, among them U1 74LVC86, U2 74LVC574, U3 74LVC574, U4 TLV74333PDBVR

Commit message: Add switch connector and slightly re-arrange xor gates
Parts:
- added JButton1: Conn_01x02, Connector_PinHeader_2.54mm:PinHeader_1x02_P2.54mm_Horizontal, symbol Connector_Generic:Conn_01x02
- R1: value 1K -> 3k3
Connections:
- wire segments 182 -> 187
- no-connect marks 23 -> 22
Other:
- moved on the sheet: U1A
Changed lines of the file:
@@
 L 74xx:74HC86 U1
 U 1 1 5F56435F
-P 8400 1500
-F 0 "U1" H 8400 1825 50  0000 C CNN
-F 1 "74LVC86" H 8400 1734 50  0000 C CNN
-F 2 "Package_SO:TSSOP-14_4.4x5mm_P0.65mm" H 8400 1500 50  0001 C CNN
-F 3 "http://www.ti.com/lit/gpn/sn74HC86" H 8400 1500 50  0001 C CNN
-	1    8400 1500
+P 8450 1500
+F 0 "U1" H 8450 1825 50  0000 C CNN
+F 1 "74LVC86" H 8450 1734 50  0000 C CNN
+F 2 "Package_SO:TSSOP-14_4.4x5mm_P0.65mm" H 8450 1500 50  0001 C CNN
+F 3 "http://www.ti.com/lit/gpn/sn74HC86" H 8450 1500 50  0001 C CNN
+	1    8450 1500
 	1    0    0    -1
 $EndComp
@@
 Connection ~ 5400 2600
 Wire Wire Line
-	7750 1500 7900 1500
-Wire Wire Line
 	5700 1000 5700 1700
 Wire Wire Line
@@
 Wire Wire Line
 	5700 1000 9700 1000
-$Comp
-L power:GND #PWR0118
-U 1 1 5F8D0C19
-P 7400 1650
-F 0 "#PWR0118" H 7400 1400 50  0001 C CNN
-F 1 "GND" H 7405 1477 50  0000 C CNN
-F 2 "" H 7400 1650 50  0001 C CNN
-F 3 "" H 7400 1650 50  0001 C CNN
-	1    7400 1650
-	1    0    0    -1
-$EndComp
-$Comp
-L power:GND #PWR0119
-U 1 1 5F8D0C4F
-P 8100 1650
-F 0 "#PWR0119" H 8100 1400 50  0001 C CNN
-F 1 "GND" H 8105 1477 50  0000 C CNN
-F 2 "" H 8100 1650 50  0001 C CNN
-F 3 "" H 8100 1650 50  0001 C CNN
-	1    8100 1650
-	1    0    0    -1
-$EndComp
-Wire Wire Line
-	8100 1650 8100 1600
-Wire Wire Line
-	8700 1500 8850 1500
+Wire Wire Line
+	8750 1500 8850 1500
 Wire Wire Line
 	8850 1500 8850 1600
@@
 Wire Wire Line
 	6900 1700 7000 1700
-Wire Wire Line
-	7000 1700 7000 1400
 Wire Wire Line
 	6900 2000 7000 2000
@@
 NoConn ~ 8800 3250
 NoConn ~ 9300 3350
-NoConn ~ 9300 4450
 NoConn ~ 8800 4550
 NoConn ~ 8800 3650
@@
 P 8150 3150
 F 0 "R1" V 7954 3150 50  0000 C CNN
-F 1 "1K" V 8045 3150 50  0000 C CNN
+F 1 "3k3" V 8045 3150 50  0000 C CNN
 F 2 "Resistor_SMD:R_0805_2012Metric_Pad1.15x1.40mm_HandSolder" H 8150 3150 50  0001 C CNN
 F 3 "~" H 8150 3150 50  0001 C CNN
@@
 Wire Wire Line
 	8250 3150 8800 3150
-NoConn ~ 8800 4350
 NoConn ~ 8800 4450
 NoConn ~ 9300 4350
@@
 Wire Wire Line
 	8000 1500 8050 1500
-Wire Wire Line
-	8050 1500 8050 1400
-Wire Wire Line
-	8050 1400 8100 1400
-Wire Wire Line
-	7400 1600 7400 1650
-Wire Wire Line
-	7000 1400 7400 1400
 Wire Wire Line
 	6900 1800 7000 1800
@@
 NoConn ~ 6900 3750
 NoConn ~ 6900 3850
+$Comp
+L power:+3.3V #PWR0107
+U 1 1 5F35F4D0
+P 7350 1350
+F 0 "#PWR0107" H 7350 1200 50  0001 C CNN
+F 1 "+3.3V" H 7365 1523 50  0000 C CNN
+F 2 "" H 7350 1350 50  0001 C CNN
+F 3 "" H 7350 1350 50  0001 C CNN
+	1    7350 1350
+	1    0    0    -1
+$EndComp
+Wire Wire Line
+	7400 1600 7000 1600
+Wire Wire Line
+	7000 1600 7000 1700
+Wire Wire Line
+	7350 1350 7350 1400
+Wire Wire Line
+	7350 1400 7400 1400
+Wire Wire Line
+	8050 1500 8050 1600
+Wire Wire Line
+	8050 1600 8150 1600
+$Comp
+L power:+3.3V #PWR0108
+U 1 1 5F39E59F
+P 8100 1350
+F 0 "#PWR0108" H 8100 1200 50  0001 C CNN
+F 1 "+3.3V" H 8115 1523 50  0000 C CNN
+F 2 "" H 8100 1350 50  0001 C CNN
+F 3 "" H 8100 1350 50  0001 C CNN
+	1    8100 1350
+	1    0    0    -1
+$EndComp
+Wire Wire Line
+	8100 1350 8100 1400
+Wire Wire Line
+	8100 1400 8150 1400
+$Comp
+L Connector_Generic:Conn_01x02 JButton1
+U 1 1 5F3EA598
+P 9950 5450
+F 0 "JButton1" V 9823 5530 50  0000 L CNN
+F 1 "Conn_01x02" V 9914 5530 50  0000 L CNN
+F 2 "Connector_PinHeader_2.54mm:PinHeader_1x02_P2.54mm_Horizontal" H 9950 5450 50  0001 C CNN
+F 3 "~" H 9950 5450 50  0001 C CNN
+	1    9950 5450
+	0    1    1    0
+$EndComp
+$Comp
+L power:GND #PWR0109
+U 1 1 5F3F766C
+P 10050 5050
+F 0 "#PWR0109" H 10050 4800 50  0001 C CNN
+F 1 "GND" V 10055 4922 50  0000 R CNN
+F 2 "" H 10050 5050 50  0001 C CNN
+F 3 "" H 10050 5050 50  0001 C CNN
+	1    10050 5050
+	0    -1   -1   0
+$EndComp
+Wire Wire Line
+	9950 5250 9950 5050
+Wire Wire Line
+	9950 5050 10050 5050
+Wire Wire Line
+	9850 5250 9850 4450
+Wire Wire Line
+	9850 4450 9300 4450
+NoConn ~ 8800 4350
 $EndSCHEMATC

Commit message: User GPIO 16 for the button. Create gerber files.
Connections:
- wire segments 187 -> 189
Changed lines of the file:
@@
 L Connector_Generic:Conn_01x02 JButton1
 U 1 1 5F3EA598
-P 9950 5450
-F 0 "JButton1" V 9823 5530 50  0000 L CNN
-F 1 "Conn_01x02" V 9914 5530 50  0000 L CNN
-F 2 "Connector_PinHeader_2.54mm:PinHeader_1x02_P2.54mm_Horizontal" H 9950 5450 50  0001 C CNN
-F 3 "~" H 9950 5450 50  0001 C CNN
-	1    9950 5450
+P 8800 5450
+F 0 "JButton1" V 8673 5530 50  0000 L CNN
+F 1 "Conn_01x02" V 8764 5530 50  0000 L CNN
+F 2 "Connector_PinHeader_2.54mm:PinHeader_1x02_P2.54mm_Horizontal" H 8800 5450 50  0001 C CNN
+F 3 "~" H 8800 5450 50  0001 C CNN
+	1    8800 5450
 	0    1    1    0
 $EndComp
@@
 L power:GND #PWR0109
 U 1 1 5F3F766C
-P 10050 5050
-F 0 "#PWR0109" H 10050 4800 50  0001 C CNN
-F 1 "GND" V 10055 4922 50  0000 R CNN
-F 2 "" H 10050 5050 50  0001 C CNN
-F 3 "" H 10050 5050 50  0001 C CNN
-	1    10050 5050
+P 8900 5050
+F 0 "#PWR0109" H 8900 4800 50  0001 C CNN
+F 1 "GND" V 8905 4922 50  0000 R CNN
+F 2 "" H 8900 5050 50  0001 C CNN
+F 3 "" H 8900 5050 50  0001 C CNN
+	1    8900 5050
 	0    -1   -1   0
 $EndComp
 Wire Wire Line
-	9950 5250 9950 5050
+	8800 5250 8800 5050
 Wire Wire Line
-	9950 5050 10050 5050
+	8800 5050 8900 5050
 Wire Wire Line
-	9850 5250 9850 4450
+	8700 5250 8700 4850
 Wire Wire Line
-	9850 4450 9300 4450
-NoConn ~ 8800 4350
+	8800 4350 8300 4350
+Wire Wire Line
+	8300 4350 8300 4850
+Wire Wire Line
+	8300 4850 8700 4850
+NoConn ~ 9300 4450
 $EndSCHEMATC
