File: kicad_AmigaAdapter/VideoSlot/V1/videoslotadapter.kicad_pcb (KiCad board)
At the start: 2 copper layers, 152 x 57.6 mm, 18 parts, among them J1 A2000 Video Slot Edge Connect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, U1 74LVC86, U2 74LVC574, U3 74LVC574, U4 TLV74333PDBVR, U5 74LVC86

Commit message: Minor CMOS fix to A2000 slot adaptor
CMOS ICs should in-general not have inputs floating. This fix ties the
unused U5 inputs high.
Parts:
- U5: footprint Housings_SSOP:TSSOP-14_4.4x5mm_Pitch0.65mm -> Package_SO:TSSOP-14_4.4x5mm_P0.65mm
- renumbered C5 to C1
Connections:
- U5 pad 10: (no net) -> +3V3
- U5 pad 11: (no net) -> Net-(U5-Pad11)
- U5 pad 12: (no net) -> +3V3
- U5 pad 13: (no net) -> +3V3
- U5 pad 8: (no net) -> Net-(U5-Pad8)
- U5 pad 9: (no net) -> +3V3
Routing:
- net +3V3: track 106.9 -> 111.9 mm
Other:
- board text added: "Adapter board for Amiga video slot V1.1 https://github.com/hoglet67"
- board text removed: "Adapter board for Amiga video slot V1.0 https://github.com/hoglet67"
