File: kicad_analog_6bit/V3/analog.sch (KiCad schematic (older format))
At the start: 35 parts, among them P1 Conn_02x06_Odd_Even, P2 Conn_01x04, P3 Conn_01x06, P6 Conn_01x01, P7 Conn_01x01, U1 MAX9108, U2 MAX9108, U3 TS12A44514DR, U4 MAX5259EEE+, U5 MCP1754S-3302xCB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

Commit message: Add IDC header for analog input
Parts:
- added P4: Conn_02x03_Odd_Even, Connector_PinHeader_2.54mm:PinHeader_2x03_P2.54mm_Horizontal, symbol Connector_Generic:Conn_02x03_Odd_Even
Changed lines of the file:
@@
 Wire Wire Line
 	4600 1750 4600 2750
+Text Label 4650 4650 2    50   ~ 0
+GND
+Text Label 4650 4750 2    50   ~ 0
+ABLUE
+Text Label 4650 4850 2    50   ~ 0
+ARED
+Text Label 5150 4650 0    50   ~ 0
+ASYNC
+Text Label 5150 4750 0    50   ~ 0
+AGREEN
+Text Label 5150 4850 0    50   ~ 0
+VCC_IN
+$Comp
+L Connector_Generic:Conn_02x03_Odd_Even P4
+U 1 1 5E55C3C0
+P 4950 4750
+F 0 "P4" H 5000 4425 50  0000 C CNN
+F 1 "Conn_02x03_Odd_Even" H 5000 4516 50  0000 C CNN
+F 2 "Connector_PinHeader_2.54mm:PinHeader_2x03_P2.54mm_Horizontal" H 4950 4750 50  0001 C CNN
+F 3 "~" H 4950 4750 50  0001 C CNN
+	1    4950 4750
+	-1   0    0    1
+$EndComp
 $EndSCHEMATC

Commit message: Update V3
Parts:
- removed P4: Conn_02x03_Odd_Even, Connector_PinHeader_2.54mm:PinHeader_2x03_P2.54mm_Horizontal, symbol Connector_Generic:Conn_02x03_Odd_Even
- added P4: Conn_01x03_ODD, Connector_Harwin:Harwin_M20-89003xx_1x03_P2.54mm_Horizontal_Custom_ODD, symbol Connector_Generic:Conn_01x03_ODD
- added P5: Conn_01x03_EVEN, Connector_Harwin:Harwin_M20-89003xx_1x03_P2.54mm_Horizontal_Custom_EVEN, symbol Connector_Generic:Conn_01x03_EVEN
- D1: footprint Diode_SMD:D_0805_2012Metric_Pad1.15x1.40mm_HandSolder -> Diode_SMD:D_SOD-123
Connections:
- net labels added: X1, X2
- net labels removed: UV1, UV2
- no-connect marks 2 -> 3
Changed lines of the file:
@@
-	1    0    0    -1
-$EndComp
-$Comp
-L Connector_Generic:Conn_01x01 P7
-U 1 1 5DD08736
-P 2150 750
-F 0 "P7" H 2230 792 50  0000 L CNN
-F 1 "Conn_01x01" H 2230 701 50  0000 L CNN
-F 2 "Connector_PinHeader_2.54mm:PinHeader_1x01_P2.54mm_Vertical" H 2150 750 50  0001 C CNN
-F 3 "~" H 2150 750 50  0001 C CNN
-	1    2150 750
 	1    0    0    -1
 $EndComp
@@
 Wire Wire Line
 	8850 2100 8850 2300
-NoConn ~ 1950 750
 NoConn ~ 1000 750
 $Comp
@@
 F 0 "D1" H 5150 1366 50  0000 C CNN
 F 1 "D_Schottky" H 5150 1275 50  0000 C CNN
-F 2 "Diode_SMD:D_0805_2012Metric_Pad1.15x1.40mm_HandSolder" H 5150 1150 50  0001 C CNN
+F 2 "Diode_SMD:D_SOD-123" H 5150 1150 50  0001 C CNN
 F 3 "~" H 5150 1150 50  0001 C CNN
 	1    5150 1150
@@
 	10700 2900 10750 2900
 Text Label 10900 4200 0    50   ~ 0
-UV1
+X1
 Text Label 10900 3100 0    50   ~ 0
-UV2
+X2
 Text Label 10150 5200 0    50   ~ 0
-UV1
+X1
 Text Label 9650 5200 2    50   ~ 0
-UV2
+X2
 Wire Wire Line
 	9100 3950 9350 3950
@@
 Wire Wire Line
 	4600 1750 4600 2750
-Text Label 4650 4650 2    50   ~ 0
+Text Label 4700 4600 2    50   ~ 0
 GND
-Text Label 4650 4750 2    50   ~ 0
+Text Label 4700 4700 2    50   ~ 0
 ABLUE
-Text Label 4650 4850 2    50   ~ 0
+Text Label 4700 4800 2    50   ~ 0
 ARED
-Text Label 5150 4650 0    50   ~ 0
+Text Label 5250 4600 0    50   ~ 0
 ASYNC
-Text Label 5150 4750 0    50   ~ 0
+Text Label 5250 4700 0    50   ~ 0
 AGREEN
-Text Label 5150 4850 0    50   ~ 0
+Text Label 5250 4800 0    50   ~ 0
 VCC_IN
 $Comp
-L Connector_Generic:Conn_02x03_Odd_Even P4
-U 1 1 5E55C3C0
-P 4950 4750
-F 0 "P4" H 5000 4425 50  0000 C CNN
-F 1 "Conn_02x03_Odd_Even" H 5000 4516 50  0000 C CNN
-F 2 "Connector_PinHeader_2.54mm:PinHeader_2x03_P2.54mm_Horizontal" H 4950 4750 50  0001 C CNN
-F 3 "~" H 4950 4750 50  0001 C CNN
-	1    4950 4750
+L Connector_Generic:Conn_01x01 P7
+U 1 1 5E6322BC
+P 2350 750
+F 0 "P7" H 2430 792 50  0000 L CNN
+F 1 "Conn_01x01" H 2430 701 50  0000 L CNN
+F 2 "Connector_PinHeader_2.54mm:PinHeader_1x01_P2.54mm_Vertical" H 2350 750 50  0001 C CNN
+F 3 "~" H 2350 750 50  0001 C CNN
+	1    2350 750
+	1    0    0    -1
+$EndComp
+NoConn ~ 2150 750
+NoConn ~ 2550 -700
+$Comp
+L Connector_Generic:Conn_01x03_EVEN P5
+U 1 1 5E57FB0D
+P 5050 4700
+F 0 "P5" H 5050 4950 50  0000 C CNN
+F 1 "Conn_01x03_EVEN" H 4750 5050 50  0000 C CNN
+F 2 "Connector_Harwin:Harwin_M20-89003xx_1x03_P2.54mm_Horizontal_Custom_EVEN" H 5050 4700 50  0001 C CNN
+F 3 "~" H 5050 4700 50  0001 C CNN
+	1    5050 4700
 	-1   0    0    1
 $EndComp
+$Comp
+L Connector_Generic:Conn_01x03_ODD P4
+U 1 1 5E580E6E
+P 4900 4700
+F 0 "P4" H 4850 4450 50  0000 L CNN
+F 1 "Conn_01x03_ODD" H 4300 4350 50  0000 L CNN
+F 2 "Connector_Harwin:Harwin_M20-89003xx_1x03_P2.54mm_Horizontal_Custom_ODD" H 4900 4700 50  0001 C CNN
+F 3 "~" H 4900 4700 50  0001 C CNN
+	1    4900 4700
+	1    0    0    -1
+$EndComp
 $EndSCHEMATC

Commit message: Update analog V3 board
Parts:
- R1: value 75R -> 100R
Changed lines of the file:
@@
 P 2400 3000
 F 0 "R1" H 2100 3050 50  0000 L CNN
-F 1 "75R" H 2100 2950 50  0000 L CNN
+F 1 "100R" H 2100 2950 50  0000 L CNN
 F 2 "Resistor_SMD:R_0805_2012Metric_Pad1.15x1.40mm_HandSolder" H 2400 3000 50  0001 C CNN
 F 3 "~" H 2400 3000 50  0001 C CNN

Commit message: Extend P4 pads on analog board
Parts:
- P3: footprint Connector_Molex:Molex_PicoBlade_53048-0610_1x06_P1.25mm_Horizontal -> Connector_Molex:Molex_PicoBlade_53048-0610_1x06_P1.25mm_Horizontal_Custom2
- P4: footprint Connector_Harwin:Harwin_M20-89003xx_1x03_P2.54mm_Horizontal_Custom_ODD -> Connector_Harwin:Harwin_M20-89003xx_1x03_P2.54mm_Horizontal_Custom_ODD2
- P5: footprint Connector_Harwin:Harwin_M20-89003xx_1x03_P2.54mm_Horizontal_Custom_EVEN -> Connector_Harwin:Harwin_M20-89003xx_1x03_P2.54mm_Horizontal_Custom_EVEN2
Changed lines of the file:
@@
 F 0 "P3" H 1368 925 50  0000 C CNN
 F 1 "Conn_01x06" H 1368 1016 50  0000 C CNN
-F 2 "Connector_Molex:Molex_PicoBlade_53048-0610_1x06_P1.25mm_Horizontal" H 1450 1450 50  0001 C CNN
+F 2 "Connector_Molex:Molex_PicoBlade_53048-0610_1x06_P1.25mm_Horizontal_Custom2" H 1450 1450 50  0001 C CNN
 F 3 "~" H 1450 1450 50  0001 C CNN
 	1    1450 1450
@@
 F 0 "P5" H 5050 4950 50  0000 C CNN
 F 1 "Conn_01x03_EVEN" H 4750 5050 50  0000 C CNN
-F 2 "Connector_Harwin:Harwin_M20-89003xx_1x03_P2.54mm_Horizontal_Custom_EVEN" H 5050 4700 50  0001 C CNN
+F 2 "Connector_Harwin:Harwin_M20-89003xx_1x03_P2.54mm_Horizontal_Custom_EVEN2" H 5050 4700 50  0001 C CNN
 F 3 "~" H 5050 4700 50  0001 C CNN
 	1    5050 4700
@@
 F 0 "P4" H 4850 4450 50  0000 L CNN
 F 1 "Conn_01x03_ODD" H 4300 4350 50  0000 L CNN
-F 2 "Connector_Harwin:Harwin_M20-89003xx_1x03_P2.54mm_Horizontal_Custom_ODD" H 4900 4700 50  0001 C CNN
+F 2 "Connector_Harwin:Harwin_M20-89003xx_1x03_P2.54mm_Horizontal_Custom_ODD2" H 4900 4700 50  0001 C CNN
 F 3 "~" H 4900 4700 50  0001 C CNN
 	1    4900 4700

Commit message: Update Analog V3 board with changed component values from wiki
Parts:
- P2: symbol Connector_Generic:Conn_01x04 -> analog-rescue:Conn_01x04-Connector_Generic
- P3: symbol Connector_Generic:Conn_01x06 -> analog-rescue:Conn_01x06-Connector_Generic
- R1: value 100R -> 470R
- U1, U2: value MAX9108 -> MAX9144; symbol analog-rescue:MAX9108-Comparator -> analog-rescue:MAX9144-Comparator-analog-rescue
- U3: value TS12A44514DR -> 74LVC4066D; symbol analog-rescue:TS12A44514DR-4xxx -> analog-rescue:74LVC4066D-4xxx-analog-rescue
- U7: value MAX9108-Comparator -> MAX9144-Comparator; symbol analog-rescue:MAX9108-Comparator -> analog-rescue:MAX9144-Comparator-analog-rescue
Changed lines of the file:
@@
 	950  7550 1250 7550
 $Comp
-L Connector_Generic:Conn_01x04 P2
+L analog-rescue:Conn_01x04-Connector_Generic P2
 U 1 1 5DCFA861
 P 750 5900
@@
 NoConn ~ 1000 750
 $Comp
-L analog-rescue:MAX9108-Comparator U2
+L analog-rescue:MAX9144-Comparator-analog-rescue U2
 U 1 1 5DD55B31
 P 9800 1250
 F 0 "U2" H 9850 1617 50  0000 C CNN
-F 1 "MAX9108" H 9850 1526 50  0000 C CNN
+F 1 "MAX9144" H 9850 1526 50  0000 C CNN
 F 2 "Package_SO:SOIC-14_3.9x8.7mm_P1.27mm" H 9500 1550 50  0001 C CNN
 F 3 "" H 9500 1550 50  0001 C CNN
@@
 $EndComp
 $Comp
-L analog-rescue:MAX9108-Comparator U2
+L analog-rescue:MAX9144-Comparator-analog-rescue U2
 U 2 1 5DD566FE
 P 9800 2000
 F 0 "U2" H 9850 2367 50  0000 C CNN
-F 1 "MAX9108" H 9850 2276 50  0000 C CNN
+F 1 "MAX9144" H 9850 2276 50  0000 C CNN
 F 2 "Package_SO:SOIC-14_3.9x8.7mm_P1.27mm" H 9500 2300 50  0001 C CNN
 F 3 "" H 9500 2300 50  0001 C CNN
@@
 $EndComp
 $Comp
-L analog-rescue:MAX9108-Comparator U2
+L analog-rescue:MAX9144-Comparator-analog-rescue U2
 U 3 1 5DD57620
 P 7300 2000
 F 0 "U2" H 7350 2367 50  0000 C CNN
-F 1 "MAX9108" H 7350 2276 50  0000 C CNN
+F 1 "MAX9144" H 7350 2276 50  0000 C CNN
 F 2 "Package_SO:SOIC-14_3.9x8.7mm_P1.27mm" H 7000 2300 50  0001 C CNN
 F 3 "" H 7000 2300 50  0001 C CNN
@@
 $EndComp
 $Comp
-L analog-rescue:MAX9108-Comparator U2
+L analog-rescue:MAX9144-Comparator-analog-rescue U2
 U 5 1 5DD583B7
 P 2850 7200
 F 0 "U2" H 2908 7296 50  0000 L CNN
-F 1 "MAX9108" H 2850 7050 50  0000 L CNN
+F 1 "MAX9144" H 2850 7050 50  0000 L CNN
 F 2 "Package_SO:SOIC-14_3.9x8.7mm_P1.27mm" H 2550 7500 50  0001 C CNN
 F 3 "" H 2550 7500 50  0001 C CNN
@@
 	2650 7450 2650 7550
 $Comp
-L analog-rescue:MAX9108-Comparator U1
+L analog-rescue:MAX9144-Comparator-analog-rescue U1
 U 2 1 5DE5166D
 P 7250 4700
 F 0 "U1" H 7300 5067 50  0000 C CNN
-F 1 "MAX9108" H 7300 4976 50  0000 C CNN
+F 1 "MAX9144" H 7300 4976 50  0000 C CNN
 F 2 "Package_SO:SOIC-14_3.9x8.7mm_P1.27mm" H 6950 5000 50  0001 C CNN
 F 3 "" H 6950 5000 50  0001 C CNN
@@
 $EndComp
 $Comp
-L analog-rescue:MAX9108-Comparator U1
+L analog-rescue:MAX9144-Comparator-analog-rescue U1
 U 1 1 5DE52F7A
 P 7250 4050
 F 0 "U1" H 7300 4417 50  0000 C CNN
-F 1 "MAX9108" H 7300 4326 50  0000 C CNN
+F 1 "MAX9144" H 7300 4326 50  0000 C CNN
 F 2 "Package_SO:SOIC-14_3.9x8.7mm_P1.27mm" H 6950 4350 50  0001 C CNN
 F 3 "" H 6950 4350 50  0001 C CNN
@@
 $EndComp
 $Comp
-L analog-rescue:MAX9108-Comparator U1
+L analog-rescue:MAX9144-Comparator-analog-rescue U1
 U 5 1 5DE550E9
 P 4250 7200
 F 0 "U1" H 4308 7296 50  0000 L CNN
-F 1 "MAX9108" H 4308 7205 50  0000 L CNN
+F 1 "MAX9144" H 4308 7205 50  0000 L CNN
 F 2 "Package_SO:SOIC-14_3.9x8.7mm_P1.27mm" H 3950 7500 50  0001 C CNN
 F 3 "" H 3950 7500 50  0001 C CNN
@@
 	6400 7550 6450 7550
 $Comp
-L analog-rescue:TS12A44514DR-4xxx U3
+L analog-rescue:74LVC4066D-4xxx-analog-rescue U3
 U 5 1 5E118FBF
 P 9050 5900
 F 0 "U3" H 9280 5946 50  0000 L CNN
-F 1 "TS12A44514DR" H 9280 5855 50  0000 L CNN
+F 1 "74LVC4066D" H 9280 5855 50  0000 L CNN
 F 2 "Package_SO:SOIC-14_3.9x8.7mm_P1.27mm" H 9050 5900 50  0001 C CNN
-F 3 "http://www.ti.com/lit/ds/symlink/cdTS12A44514DRb.pdf" H 9050 5900 50  0001 C CNN
+F 3 "http://www.ti.com/lit/ds/symlink/cd74LVC4066Db.pdf" H 9050 5900 50  0001 C CNN
 	5    9050 5900
 	1    0    0    -1
@@
 GND
 $Comp
-L analog-rescue:TS12A44514DR-4xxx U3
+L analog-rescue:74LVC4066D-4xxx-analog-rescue U3
 U 1 1 5E1234E2
 P 2400 3550
 F 0 "U3" V 2150 3950 50  0000 R CNN
-F 1 "TS12A44514DR" V 2250 4250 50  0000 R CNN
+F 1 "74LVC4066D" V 2250 4250 50  0000 R CNN
 F 2 "Package_SO:SOIC-14_3.9x8.7mm_P1.27mm" H 2400 3550 50  0001 C CNN
-F 3 "http://www.ti.com/lit/ds/symlink/cdTS12A44514DRb.pdf" H 2400 3550 50  0001 C CNN
+F 3 "http://www.ti.com/lit/ds/symlink/cd74LVC4066Db.pdf" H 2400 3550 50  0001 C CNN
 	1    2400 3550
 	0    -1   1    0
 $EndComp
 $Comp
-L analog-rescue:TS12A44514DR-4xxx U3
+L analog-rescue:74LVC4066D-4xxx-analog-rescue U3
 U 2 1 5E127744
 P 4600 3550
 F 0 "U3" V 4800 3950 50  0000 R CNN
-F 1 "TS12A44514DR" V 4900 4150 50  0000 R CNN
+F 1 "74LVC4066D" V 4900 4150 50  0000 R CNN
 F 2 "Package_SO:SOIC-14_3.9x8.7mm_P1.27mm" H 4600 3550 50  0001 C CNN
-F 3 "http://www.ti.com/lit/ds/symlink/cdTS12A44514DRb.pdf" H 4600 3550 50  0001 C CNN
+F 3 "http://www.ti.com/lit/ds/symlink/cd74LVC4066Db.pdf" H 4600 3550 50  0001 C CNN
 	2    4600 3550
 	0    1    1    0
 $EndComp
 $Comp
-L analog-rescue:TS12A44514DR-4xxx U3
+L analog-rescue:74LVC4066D-4xxx-analog-rescue U3
 U 3 1 5E129BF6
 P 3150 3550
 F 0 "U3" V 3350 3300 50  0000 R CNN
-F 1 "TS12A44514DR" V 3450 3500 50  0000 R CNN
+F 1 "74LVC4066D" V 3450 3500 50  0000 R CNN
 F 2 "Package_SO:SOIC-14_3.9x8.7mm_P1.27mm" H 3150 3550 50  0001 C CNN
-F 3 "http://www.ti.com/lit/ds/symlink/cdTS12A44514DRb.pdf" H 3150 3550 50  0001 C CNN
+F 3 "http://www.ti.com/lit/ds/symlink/cd74LVC4066Db.pdf" H 3150 3550 50  0001 C CNN
 	3    3150 3550
 	0    1    1    0
@@
 P 2400 3000
 F 0 "R1" H 2100 3050 50  0000 L CNN
-F 1 "100R" H 2100 2950 50  0000 L CNN
+F 1 "470R" H 2100 2950 50  0000 L CNN
 F 2 "Resistor_SMD:R_0805_2012Metric_Pad1.15x1.40mm_HandSolder" H 2400 3000 50  0001 C CNN
 F 3 "~" H 2400 3000 50  0001 C CNN
@@
 	1650 1550 2250 1550
 $Comp
-L analog-rescue:MAX9108-Comparator U2
+L analog-rescue:MAX9144-Comparator-analog-rescue U2
 U 4 1 5DD54DB9
 P 7300 1250
 F 0 "U2" H 7350 1617 50  0000 C CNN
-F 1 "MAX9108" H 7350 1526 50  0000 C CNN
+F 1 "MAX9144" H 7350 1526 50  0000 C CNN
 F 2 "Package_SO:SOIC-14_3.9x8.7mm_P1.27mm" H 7000 1550 50  0001 C CNN
 F 3 "" H 7000 1550 50  0001 C CNN
@@
 $EndComp
 $Comp
-L analog-rescue:MAX9108-Comparator U1
+L analog-rescue:MAX9144-Comparator-analog-rescue U1
 U 4 1 5DE53BEC
 P 7250 3400
 F 0 "U1" H 7300 3767 50  0000 C CNN
-F 1 "MAX9108" H 7300 3676 50  0000 C CNN
+F 1 "MAX9144" H 7300 3676 50  0000 C CNN
 F 2 "Package_SO:SOIC-14_3.9x8.7mm_P1.27mm" H 6950 3700 50  0001 C CNN
 F 3 "" H 6950 3700 50  0001 C CNN
@@
 Connection ~ 2250 6850
 $Comp
-L Connector_Generic:Conn_01x06 P3
+L analog-rescue:Conn_01x06-Connector_Generic P3
 U 1 1 5E3F9F6C
 P 1450 1450
@@
 	1650 4850 1650 5000
 $Comp
-L analog-rescue:TS12A44514DR-4xxx U3
+L analog-rescue:74LVC4066D-4xxx-analog-rescue U3
 U 4 1 5E12E54E
 P 3900 3550
 F 0 "U3" V 4100 3250 50  0000 R CNN
-F 1 "TS12A44514DR" V 4200 3450 50  0000 R CNN
+F 1 "74LVC4066D" V 4200 3450 50  0000 R CNN
 F 2 "Package_SO:SOIC-14_3.9x8.7mm_P1.27mm" H 3900 3550 50  0001 C CNN
-F 3 "http://www.ti.com/lit/ds/symlink/cdTS12A44514DRb.pdf" H 3900 3550 50  0001 C CNN
+F 3 "http://www.ti.com/lit/ds/symlink/cd74LVC4066Db.pdf" H 3900 3550 50  0001 C CNN
 	4    3900 3550
 	0    1    1    0
@@
 	7000 5450 6950 5450
 $Comp
-L analog-rescue:MAX9108-Comparator U1
+L analog-rescue:MAX9144-Comparator-analog-rescue U1
 U 3 1 5DE522AE
 P 7250 5550
 F 0 "U1" H 7300 5917 50  0000 C CNN
-F 1 "MAX9108" H 7300 5826 50  0000 C CNN
+F 1 "MAX9144" H 7300 5826 50  0000 C CNN
 F 2 "Package_SO:SOIC-14_3.9x8.7mm_P1.27mm" H 6950 5850 50  0001 C CNN
 F 3 "" H 6950 5850 50  0001 C CNN
@@
 ASYNC
 $Comp
-L analog-rescue:MAX9108-Comparator U7
+L analog-rescue:MAX9144-Comparator-analog-rescue U7
 U 4 1 5E591929
 P 10350 2900
 F 0 "U7" H 10000 3250 50  0000 C CNN
-F 1 "MAX9108-Comparator" H 10100 3150 50  0000 C CNN
+F 1 "MAX9144-Comparator" H 10100 3150 50  0000 C CNN
 F 2 "Package_SO:SOIC-14_3.9x8.7mm_P1.27mm" H 10050 3200 50  0001 C CNN
 F 3 "" H 10050 3200 50  0001 C CNN
@@
 $EndComp
 $Comp
-L analog-rescue:MAX9108-Comparator U7
+L analog-rescue:MAX9144-Comparator-analog-rescue U7
 U 5 1 5E592994
 P 9900 6000
 F 0 "U7" H 9800 5850 50  0000 C CNN
-F 1 "MAX9108-Comparator" H 9750 5500 50  0000 C CNN
+F 1 "MAX9144-Comparator" H 9750 5500 50  0000 C CNN
 F 2 "Package_SO:SOIC-14_3.9x8.7mm_P1.27mm" H 9600 6300 50  0001 C CNN
 F 3 "" H 9600 6300 50  0001 C CNN
@@
 $EndComp
 $Comp
-L analog-rescue:MAX9108-Comparator U7
+L analog-rescue:MAX9144-Comparator-analog-rescue U7
 U 1 1 5E593759
 P 8750 2850
 F 0 "U7" H 8800 3217 50  0000 C CNN
-F 1 "MAX9108-Comparator" H 8800 3126 50  0000 C CNN
+F 1 "MAX9144-Comparator" H 8800 3126 50  0000 C CNN
 F 2 "Package_SO:SOIC-14_3.9x8.7mm_P1.27mm" H 8450 3150 50  0001 C CNN
 F 3 "" H 8450 3150 50  0001 C CNN
@@
 $EndComp
 $Comp
-L analog-rescue:MAX9108-Comparator U7
+L analog-rescue:MAX9144-Comparator-analog-rescue U7
 U 2 1 5E5947A9
 P 8750 3950
 F 0 "U7" H 8800 4350 50  0000 C CNN
-F 1 "MAX9108-Comparator" H 8800 4226 50  0000 C CNN
+F 1 "MAX9144-Comparator" H 8800 4226 50  0000 C CNN
 F 2 "Package_SO:SOIC-14_3.9x8.7mm_P1.27mm" H 8450 4250 50  0001 C CNN
 F 3 "" H 8450 4250 50  0001 C CNN
@@
 $EndComp
 $Comp
-L analog-rescue:MAX9108-Comparator U7
+L analog-rescue:MAX9144-Comparator-analog-rescue U7
 U 3 1 5E5959CE
 P 10350 4000
 F 0 "U7" H 10350 4500 50  0000 L CNN
-F 1 "MAX9108-Comparator" H 10050 4400 50  0000 L CNN
+F 1 "MAX9144-Comparator" H 10050 4400 50  0000 L CNN
 F 2 "Package_SO:SOIC-14_3.9x8.7mm_P1.27mm" H 10050 4300 50  0001 C CNN
 F 3 "" H 10050 4300 50  0001 C CNN

Commit message: Moved most component values from the Fab. Layer to the Silk Layer on the analog board and the 12-bit board to serve as an aid when placing the componets during assembly.
Generated interactive Bill Of Materials for the analog board and the 12-bit board to serve as an aid when
sourcing components and assembly.These are in the "bom" directory.

Replaced the Gerber files for the analog board and the 12-bit board with the updated silk screens.
Parts:
- P4: symbol Connector_Generic:Conn_01x03_ODD -> analog-rescue:Conn_01x03_ODD-Connector_Generic
- P5: symbol Connector_Generic:Conn_01x03_EVEN -> analog-rescue:Conn_01x03_EVEN-Connector_Generic
- U4: symbol Analog_DAC:MAX5259EEE+ -> analog-rescue:MAX5259EEE+-Analog_DAC
Changed lines of the file:
@@
 EESchema Schematic File Version 4
-LIBS:analog-cache
 EELAYER 30 0
 EELAYER END
@@
 	3650 7550 4050 7550
 $Comp
-L Analog_DAC:MAX5259EEE+ U4
+L analog-rescue:MAX5259EEE+-Analog_DAC U4
 U 1 1 5DEBF7A0
 P 2400 5900
@@
 NoConn ~ 2550 -700
 $Comp
-L Connector_Generic:Conn_01x03_EVEN P5
+L analog-rescue:Conn_01x03_EVEN-Connector_Generic P5
 U 1 1 5E57FB0D
 P 5050 4700
@@
 $EndComp
 $Comp
-L Connector_Generic:Conn_01x03_ODD P4
+L analog-rescue:Conn_01x03_ODD-Connector_Generic P4
 U 1 1 5E580E6E
 P 4900 4700
